Commit message: robot can move

File: ros/src/robot_simulation/urdf/robot_simulation.xacro (robot description, xacro)
@@ -1,10 +1,4 @@
 <?xml version="1.0"?>
 <robot xmlns:xacro="http://www.ros.org/wiki/xacro" name="robot_simulation">
-  <gazebo reference="right_wheel">
-    <material>Gazebo/Blue</material>
-  </gazebo>
-  <gazebo reference="left_wheel">
-    <material>Gazebo/Blue</material>
-  </gazebo>
   <link name="base_link">
     <inertial>
@@ -73,4 +67,13 @@
     <axis xyz="0.0 1 0.0"/>
   </joint>
+  <transmission name="right_wheel_trans">
+    <type>transmission_interface/SimpleTransmission</type>
+    <joint name="right_joint">
+        <hardwareInterface>VelocityJointInterface</hardwareInterface>
+    </joint>
+    <actuator name="right_motor">
+        <mechanicalReduction>1.0</mechanicalReduction>
+    </actuator>
+  </transmission>
   <link name="left_wheel">
     <inertial>
@@ -97,4 +100,27 @@
     <axis xyz="0.0 1 0.0"/>
   </joint>
+  <transmission name="left_wheel_trans">
+    <type>transmission_interface/SimpleTransmission</type>
+    <joint name="left_joint">
+        <hardwareInterface>VelocityJointInterface</hardwareInterface>
+    </joint>
+    <actuator name="left_motor">
+        <mechanicalReduction>1.0</mechanicalReduction>
+    </actuator>
+  </transmission>
+  <gazebo reference="right_wheel">
+      <mu1 value="200.0"/>
+      <mu2 value="100.0"/>
+      <kp value="10000000.0" />
+      <kd value="1.0" />
+      <material>Gazebo/Blue</material>
+  </gazebo>
+  <gazebo reference="left_wheel">
+      <mu1 value="200.0"/>
+      <mu2 value="100.0"/>
+      <kp value="10000000.0" />
+      <kd value="1.0" />
+      <material>Gazebo/Blue</material>
+  </gazebo>
   <!-- Gazebo plugin for ROS Control -->
   <gazebo>

Commit message: added a script for moving a robot

File: ros/src/robot_simulation/urdf/robot_simulation.xacro (robot description, xacro)
@@ -62,5 +62,5 @@
   </link>
   <joint name="right_joint" type="continuous">
-    <origin xyz="0.0 0.226 0.1" rpy="0.0 0.0 0.0"/>
+    <origin xyz="0.0 -0.226 0.1" rpy="0.0 0.0 0.0"/>
     <parent link="base_link"/>
     <child link="right_wheel"/>
@@ -95,5 +95,5 @@
   </link>
   <joint name="left_joint" type="continuous">
-    <origin xyz="0.0 -0.226 0.1" rpy="0.0 0.0 0.0"/>
+    <origin xyz="0.0 0.226 0.1" rpy="0.0 0.0 0.0"/>
     <parent link="base_link"/>
     <child link="left_wheel"/>

Commit message: changed the urdf robot model

File: ros/src/robot_simulation/urdf/robot_simulation.xacro (robot description, xacro)
@@ -7,46 +7,22 @@
     </inertial>
     <visual name="base_visual">
-      <origin xyz="0.0 0.0 0.15" rpy="0.0 0.0 0.0"/>
+      <origin xyz="0.0 0.0 0.1" rpy="0.0 0.0 0.0"/>
       <geometry>
-        <cylinder length="0.2" radius="0.2"/>
+        <box size="0.6 0.4 0.1"/>
       </geometry>
     </visual>
     <collision name="base_collision">
-      <origin xyz="0.0 0.0 0.15" rpy="0.0 0.0 0.0"/>
+      <origin xyz="0.0 0.0 0.1" rpy="0.0 0.0 0.0"/>
       <geometry>
-        <cylinder length="0.2" radius="0.2"/>
+        <box size="0.6 0.4 0.1"/>
       </geometry>
     </collision>
-    <visual name="front_sphere_visual">
-        <origin xyz="0.15 0.0 0.05" rpy="0.0 0.0 0.0"/>
-        <geometry>
-            <sphere radius="0.0499"/>
-        </geometry>
-    </visual>
-    <collision name="front_sphere_collision">
-        <origin xyz="0.15 0.0 0.05" rpy="0.0 0.0 0.0"/>
-        <geometry>
-            <sphere radius="0.0499"/>
-        </geometry>
-    </collision>
-    <visual name="back_sphere_visual">
-        <origin xyz="-0.15 0.0 0.05" rpy="0.0 0.0 0.0"/>
-        <geometry>
-            <sphere radius="0.0499"/>
-        </geometry>
-    </visual>
-    <collision name="back_sphere_collision">
-        <origin xyz="-0.15 0.0 0.05" rpy="0.0 0.0 0.0"/>
-        <geometry>
-            <sphere radius="0.0499"/>
-        </geometry>
-    </collision>
   </link>
-  <link name="right_wheel">
+  <link name="right_front_wheel">
     <inertial>
         <mass value="5.0"/>
         <inertia ixx="1.0" ixy="0.0" ixz="0.0" iyy="1.0" iyz="0.0" izz="1.0"/>
     </inertial>
-    <visual name="right_wheel_visual">
+    <visual name="right_front_wheel_visual">
         <origin xyz="0.0 0.0 0.0" rpy="1.57075 0 0"/>
         <geometry>
@@ -54,5 +30,5 @@
         </geometry>
     </visual>
-    <collision name="right_wheel_collision">
+    <collision name="right_front_wheel_collision">
         <origin xyz="0.0 0.0 0.0" rpy="1.57075 0 0"/>
         <geometry>
@@ -61,25 +37,10 @@
     </collision>
   </link>
-  <joint name="right_joint" type="continuous">
-    <origin xyz="0.0 -0.226 0.1" rpy="0.0 0.0 0.0"/>
-    <parent link="base_link"/>
-    <child link="right_wheel"/>
-    <axis xyz="0.0 1 0.0"/>
-  </joint>
-  <transmission name="right_wheel_trans">
-    <type>transmission_interface/SimpleTransmission</type>
-    <joint name="right_joint">
-        <hardwareInterface>VelocityJointInterface</hardwareInterface>
-    </joint>
-    <actuator name="right_motor">
-        <mechanicalReduction>1.0</mechanicalReduction>
-    </actuator>
-  </transmission>
-  <link name="left_wheel">
+  <link name="right_back_wheel">
     <inertial>
         <mass value="5.0"/>
         <inertia ixx="1.0" ixy="0.0" ixz="0.0" iyy="1.0" iyz="0.0" izz="1.0"/>
     </inertial>
-    <visual name="left_wheel_visual">
+    <visual name="right_back_wheel_visual">
         <origin xyz="0.0 0.0 0.0" rpy="1.57075 0 0"/>
         <geometry>
@@ -87,5 +48,5 @@
         </geometry>
     </visual>
-    <collision name="left_wheel_collision">
+    <collision name="right_back_wheel_collision">
         <origin xyz="0.0 0.0 0.0" rpy="1.57075 0 0"/>
         <geometry>
@@ -94,20 +55,101 @@
     </collision>
   </link>
-  <joint name="left_joint" type="continuous">
-    <origin xyz="0.0 0.226 0.1" rpy="0.0 0.0 0.0"/>
+  <joint name="right_front_joint" type="continuous">
+    <origin xyz="0.15 -0.226 0.1" rpy="0.0 0.0 0.0"/>
     <parent link="base_link"/>
-    <child link="left_wheel"/>
+    <child link="right_front_wheel"/>
     <axis xyz="0.0 1 0.0"/>
   </joint>
-  <transmission name="left_wheel_trans">
+  <joint name="right_back_joint" type="continuous">
+    <origin xyz="-0.15 -0.226 0.1" rpy="0.0 0.0 0.0"/>
+    <parent link="base_link"/>
+    <child link="right_back_wheel"/>
+    <axis xyz="0.0 1 0.0"/>
+  </joint>
+  <transmission name="right_front_wheel_trans">
     <type>transmission_interface/SimpleTransmission</type>
-    <joint name="left_joint">
+    <joint name="right_front_joint">
         <hardwareInterface>VelocityJointInterface</hardwareInterface>
     </joint>
-    <actuator name="left_motor">
+    <actuator name="right_front_motor">
         <mechanicalReduction>1.0</mechanicalReduction>
     </actuator>
   </transmission>
-  <gazebo reference="right_wheel">
+  <transmission name="right_back_wheel_trans">
+    <type>transmission_interface/SimpleTransmission</type>
+    <joint name="right_back_joint">
+        <hardwareInterface>VelocityJointInterface</hardwareInterface>
+    </joint>
+    <actuator name="right_back_motor">
+        <mechanicalReduction>1.0</mechanicalReduction>
+    </actuator>
+  </transmission>
+  <link name="left_front_wheel">
+    <inertial>
+        <mass value="5.0"/>
+        <inertia ixx="1.0" ixy="0.0" ixz="0.0" iyy="1.0" iyz="0.0" izz="1.0"/>
+    </inertial>
+    <visual name="left_front_wheel_visual">
+        <origin xyz="0.0 0.0 0.0" rpy="1.57075 0 0"/>
+        <geometry>
+            <cylinder radius="0.1" length="0.05"/>
+        </geometry>
+    </visual>
+    <collision name="left_front_wheel_collision">
+        <origin xyz="0.0 0.0 0.0" rpy="1.57075 0 0"/>
+        <geometry>
+            <cylinder radius="0.1" length="0.05"/>
+        </geometry>
+    </collision>
+  </link>
+  <link name="left_back_wheel">
+    <inertial>
+        <mass value="5.0"/>
+        <inertia ixx="1.0" ixy="0.0" ixz="0.0" iyy="1.0" iyz="0.0" izz="1.0"/>
+    </inertial>
+    <visual name="left_back_wheel_visual">
+        <origin xyz="0.0 0.0 0.0" rpy="1.57075 0 0"/>
+        <geometry>
+            <cylinder radius="0.1" length="0.05"/>
+        </geometry>
+    </visual>
+    <collision name="left_back_wheel_collision">
+        <origin xyz="0.0 0.0 0.0" rpy="1.57075 0 0"/>
+        <geometry>
+            <cylinder radius="0.1" length="0.05"/>
+        </geometry>
+    </collision>
+  </link>
+  <joint name="left_front_joint" type="continuous">
+    <origin xyz="0.15 0.226 0.1" rpy="0.0 0.0 0.0"/>
+    <parent link="base_link"/>
+    <child link="left_front_wheel"/>
+    <axis xyz="0.0 1 0.0"/>
+  </joint>
+  <joint name="left_back_joint" type="continuous">
+    <origin xyz="-0.15 0.226 0.1" rpy="0.0 0.0 0.0"/>
+    <parent link="base_link"/>
+    <child link="left_back_wheel"/>
+    <axis xyz="0.0 1 0.0"/>
+  </joint>
+  <transmission name="left_front_wheel_trans">
+    <type>transmission_interface/SimpleTransmission</type>
+    <joint name="left_front_joint">
+        <hardwareInterface>VelocityJointInterface</hardwareInterface>
+    </joint>
+    <actuator name="left_front_motor">
+        <mechanicalReduction>1.0</mechanicalReduction>
+    </actuator>
+  </transmission>
+  <transmission name="left_back_wheel_trans">
+    <type>transmission_interface/SimpleTransmission</type>
+    <joint name="left_back_joint">
+        <hardwareInterface>VelocityJointInterface</hardwareInterface>
+    </joint>
+    <actuator name="left_back_motor">
+        <mechanicalReduction>1.0</mechanicalReduction>
+    </actuator>
+  </transmission>
+  <gazebo reference="right_front_wheel">
       <mu1 value="200.0"/>
       <mu2 value="100.0"/>
@@ -116,5 +158,19 @@
       <material>Gazebo/Blue</material>
   </gazebo>
-  <gazebo reference="left_wheel">
+  <gazebo reference="right_back_wheel">
+      <mu1 value="200.0"/>
+      <mu2 value="100.0"/>
+      <kp value="10000000.0" />
+      <kd value="1.0" />
+      <material>Gazebo/Blue</material>
+  </gazebo>
+  <gazebo reference="left_front_wheel">
+      <mu1 value="200.0"/>
+      <mu2 value="100.0"/>
+      <kp value="10000000.0" />
+      <kd value="1.0" />
+      <material>Gazebo/Blue</material>
+  </gazebo>
+  <gazebo reference="left_back_wheel">
       <mu1 value="200.0"/>
       <mu2 value="100.0"/>

Commit message: added a wheel description macro in xacro file

File: ros/src/robot_simulation/urdf/robot_simulation.xacro (robot description, xacro)
@@ -1,4 +1,30 @@
 <?xml version="1.0"?>
 <robot xmlns:xacro="http://www.ros.org/wiki/xacro" name="robot_simulation">
+  <xacro:macro name="base_geometry">
+    <origin xyz="0.0 0.0 0.1" rpy="0.0 0.0 0.0"/>
+      <geometry>
+        <box size="0.6 0.4 0.1"/>
+      </geometry>
+  </xacro:macro>
+  <xacro:macro name="wheel_description" params="name">
+    <link name="${name}">
+    <inertial>
+        <mass value="5.0"/>
+        <inertia ixx="1.0" ixy="0.0" ixz="0.0" iyy="1.0" iyz="0.0" izz="1.0"/>
+    </inertial>
+    <visual>
+        <origin xyz="0.0 0.0 0.0" rpy="1.57075 0 0"/>
+        <geometry>
+            <cylinder radius="0.1" length="0.05"/>
+        </geometry>
+    </visual>
+    <collision>
+        <origin xyz="0.0 0.0 0.0" rpy="1.57075 0 0"/>
+        <geometry>
+            <cylinder radius="0.1" length="0.05"/>
+        </geometry>
+    </collision>
+  </link>
+  </xacro:macro>
   <link name="base_link">
     <inertial>
@@ -7,52 +33,12 @@
     </inertial>
     <visual name="base_visual">
-      <origin xyz="0.0 0.0 0.1" rpy="0.0 0.0 0.0"/>
-      <geometry>
-        <box size="0.6 0.4 0.1"/>
-      </geometry>
+      <xacro:base_geometry />
     </visual>
     <collision name="base_collision">
-      <origin xyz="0.0 0.0 0.1" rpy="0.0 0.0 0.0"/>
-      <geometry>
-        <box size="0.6 0.4 0.1"/>
-      </geometry>
+      <xacro:base_geometry />
     </collision>
   </link>
-  <link name="right_front_wheel">
-    <inertial>
-        <mass value="5.0"/>
-        <inertia ixx="1.0" ixy="0.0" ixz="0.0" iyy="1.0" iyz="0.0" izz="1.0"/>
-    </inertial>
-    <visual name="right_front_wheel_visual">
-        <origin xyz="0.0 0.0 0.0" rpy="1.57075 0 0"/>
-        <geometry>
-            <cylinder radius="0.1" length="0.05"/>
-        </geometry>
-    </visual>
-    <collision name="right_front_wheel_collision">
-        <origin xyz="0.0 0.0 0.0" rpy="1.57075 0 0"/>
-        <geometry>
-            <cylinder radius="0.1" length="0.05"/>
-        </geometry>
-    </collision>
-  </link>
-  <link name="right_back_wheel">
-    <inertial>
-        <mass value="5.0"/>
-        <inertia ixx="1.0" ixy="0.0" ixz="0.0" iyy="1.0" iyz="0.0" izz="1.0"/>
-    </inertial>
-    <visual name="right_back_wheel_visual">
-        <origin xyz="0.0 0.0 0.0" rpy="1.57075 0 0"/>
-        <geometry>
-            <cylinder radius="0.1" length="0.05"/>
-        </geometry>
-    </visual>
-    <collision name="right_back_wheel_collision">
-        <origin xyz="0.0 0.0 0.0" rpy="1.57075 0 0"/>
-        <geometry>
-            <cylinder radius="0.1" length="0.05"/>
-        </geometry>
-    </collision>
-  </link>
+  <xacro:wheel_description name="right_front_wheel" />
+  <xacro:wheel_description name="right_back_wheel" />
   <joint name="right_front_joint" type="continuous">
     <origin xyz="0.15 -0.226 0.1" rpy="0.0 0.0 0.0"/>
@@ -85,40 +71,6 @@
     </actuator>
   </transmission>
-  <link name="left_front_wheel">
-    <inertial>
-        <mass value="5.0"/>
-        <inertia ixx="1.0" ixy="0.0" ixz="0.0" iyy="1.0" iyz="0.0" izz="1.0"/>
-    </inertial>
-    <visual name="left_front_wheel_visual">
-        <origin xyz="0.0 0.0 0.0" rpy="1.57075 0 0"/>
-        <geometry>
-            <cylinder radius="0.1" length="0.05"/>
-        </geometry>
-    </visual>
-    <collision name="left_front_wheel_collision">
-        <origin xyz="0.0 0.0 0.0" rpy="1.57075 0 0"/>
-        <geometry>
-            <cylinder radius="0.1" length="0.05"/>
-        </geometry>
-    </collision>
-  </link>
-  <link name="left_back_wheel">
-    <inertial>
-        <mass value="5.0"/>
-        <inertia ixx="1.0" ixy="0.0" ixz="0.0" iyy="1.0" iyz="0.0" izz="1.0"/>
-    </inertial>
-    <visual name="left_back_wheel_visual">
-        <origin xyz="0.0 0.0 0.0" rpy="1.57075 0 0"/>
-        <geometry>
-            <cylinder radius="0.1" length="0.05"/>
-        </geometry>
-    </visual>
-    <collision name="left_back_wheel_collision">
-        <origin xyz="0.0 0.0 0.0" rpy="1.57075 0 0"/>
-        <geometry>
-            <cylinder radius="0.1" length="0.05"/>
-        </geometry>
-    </collision>
-  </link>
+  <xacro:wheel_description name="left_front_wheel" />
+  <xacro:wheel_description name="left_back_wheel" />
   <joint name="left_front_joint" type="continuous">
     <origin xyz="0.15 0.226 0.1" rpy="0.0 0.0 0.0"/>

Commit message: added macros of redundant descriptions in a xacro file

File: ros/src/robot_simulation/urdf/robot_simulation.xacro (robot description, xacro)
@@ -1,4 +1,5 @@
 <?xml version="1.0"?>
 <robot xmlns:xacro="http://www.ros.org/wiki/xacro" name="robot_simulation">
+  <!-- begin macros definition -->
   <xacro:macro name="base_geometry">
     <origin xyz="0.0 0.0 0.1" rpy="0.0 0.0 0.0"/>
@@ -27,4 +28,33 @@
   </link>
   </xacro:macro>
+  <xacro:macro name="joint_desc" params="side side2 x y">
+    <joint name="${side}_${side2}_joint" type="continuous">
+      <origin xyz="${x} ${y} 0.1" rpy="0.0 0.0 0.0"/>
+      <parent link="base_link"/>
+      <child link="${side}_${side2}_wheel"/>
+      <axis xyz="0.0 1 0.0"/>
+    </joint>
+  </xacro:macro>
+  <xacro:macro name="transmission_desc" params="side side2">
+    <transmission name="${side}_${side2}_wheel_trans">
+      <type>transmission_interface/SimpleTransmission</type>
+      <joint name="${side}_${side2}_joint">
+        <hardwareInterface>VelocityJointInterface</hardwareInterface>
+      </joint>
+      <actuator name="${side}_${side2}_motor">
+        <mechanicalReduction>1.0</mechanicalReduction>
+      </actuator>
+    </transmission>
+  </xacro:macro>
+  <xacro:macro name="gazebo_wheel" params="ref">
+    <gazebo reference="${ref}">
+      <mu1 value="200.0"/>
+      <mu2 value="100.0"/>
+      <kp value="10000000.0" />
+      <kd value="1.0" />
+      <material>Gazebo/Blue</material>
+    </gazebo>
+  </xacro:macro>
+  <!-- end macros definition -->
   <link name="base_link">
     <inertial>
@@ -41,94 +71,18 @@
   <xacro:wheel_description name="right_front_wheel" />
   <xacro:wheel_description name="right_back_wheel" />
-  <joint name="right_front_joint" type="continuous">
-    <origin xyz="0.15 -0.226 0.1" rpy="0.0 0.0 0.0"/>
-    <parent link="base_link"/>
-    <child link="right_front_wheel"/>
-    <axis xyz="0.0 1 0.0"/>
-  </joint>
-  <joint name="right_back_joint" type="continuous">
-    <origin xyz="-0.15 -0.226 0.1" rpy="0.0 0.0 0.0"/>
-    <parent link="base_link"/>
-    <child link="right_back_wheel"/>
-    <axis xyz="0.0 1 0.0"/>
-  </joint>
-  <transmission name="right_front_wheel_trans">
-    <type>transmission_interface/SimpleTransmission</type>
-    <joint name="right_front_joint">
-        <hardwareInterface>VelocityJointInterface</hardwareInterface>
-    </joint>
-    <actuator name="right_front_motor">
-        <mechanicalReduction>1.0</mechanicalReduction>
-    </actuator>
-  </transmission>
-  <transmission name="right_back_wheel_trans">
-    <type>transmission_interface/SimpleTransmission</type>
-    <joint name="right_back_joint">
-        <hardwareInterface>VelocityJointInterface</hardwareInterface>
-    </joint>
-    <actuator name="right_back_motor">
-        <mechanicalReduction>1.0</mechanicalReduction>
-    </actuator>
-  </transmission>
   <xacro:wheel_description name="left_front_wheel" />
   <xacro:wheel_description name="left_back_wheel" />
-  <joint name="left_front_joint" type="continuous">
-    <origin xyz="0.15 0.226 0.1" rpy="0.0 0.0 0.0"/>
-    <parent link="base_link"/>
-    <child link="left_front_wheel"/>
-    <axis xyz="0.0 1 0.0"/>
-  </joint>
-  <joint name="left_back_joint" type="continuous">
-    <origin xyz="-0.15 0.226 0.1" rpy="0.0 0.0 0.0"/>
-    <parent link="base_link"/>
-    <child link="left_back_wheel"/>
-    <axis xyz="0.0 1 0.0"/>
-  </joint>
-  <transmission name="left_front_wheel_trans">
-    <type>transmission_interface/SimpleTransmission</type>
-    <joint name="left_front_joint">
-        <hardwareInterface>VelocityJointInterface</hardwareInterface>
-    </joint>
-    <actuator name="left_front_motor">
-        <mechanicalReduction>1.0</mechanicalReduction>
-    </actuator>
-  </transmission>
-  <transmission name="left_back_wheel_trans">
-    <type>transmission_interface/SimpleTransmission</type>
-    <joint name="left_back_joint">
-        <hardwareInterface>VelocityJointInterface</hardwareInterface>
-    </joint>
-    <actuator name="left_back_motor">
-        <mechanicalReduction>1.0</mechanicalReduction>
-    </actuator>
-  </transmission>
-  <gazebo reference="right_front_wheel">
-      <mu1 value="200.0"/>
-      <mu2 value="100.0"/>
-      <kp value="10000000.0" />
-      <kd value="1.0" />
-      <material>Gazebo/Blue</material>
-  </gazebo>
-  <gazebo reference="right_back_wheel">
-      <mu1 value="200.0"/>
-      <mu2 value="100.0"/>
-      <kp value="10000000.0" />
-      <kd value="1.0" />
-      <material>Gazebo/Blue</material>
-  </gazebo>
-  <gazebo reference="left_front_wheel">
-      <mu1 value="200.0"/>
-      <mu2 value="100.0"/>
-      <kp value="10000000.0" />
-      <kd value="1.0" />
-      <material>Gazebo/Blue</material>
-  </gazebo>
-  <gazebo reference="left_back_wheel">
-      <mu1 value="200.0"/>
-      <mu2 value="100.0"/>
-      <kp value="10000000.0" />
-      <kd value="1.0" />
-      <material>Gazebo/Blue</material>
-  </gazebo>
+  <xacro:joint_desc side="right" side2="front" x="0.15" y="-0.226" />
+  <xacro:joint_desc side="right" side2="back" x="-0.15" y="-0.226" />
+  <xacro:joint_desc side="left" side2="front" x="0.15" y="0.226" />
+  <xacro:joint_desc side="left" side2="back" x="-0.15" y="0.226" />
+  <xacro:transmission_desc side="right" side2="front" />
+  <xacro:transmission_desc side="right" side2="back" />
+  <xacro:transmission_desc side="left" side2="front" />
+  <xacro:transmission_desc side="left" side2="back" />
+  <xacro:gazebo_wheel ref="right_front_wheel" />
+  <xacro:gazebo_wheel ref="right_back_wheel" />
+  <xacro:gazebo_wheel ref="left_front_wheel" />
+  <xacro:gazebo_wheel ref="left_back_wheel" />
   <!-- Gazebo plugin for ROS Control -->
   <gazebo>

Commit message: added an accelerometer to the urdf model

File: ros/src/robot_simulation/urdf/robot_simulation.xacro (robot description, xacro)
@@ -85,4 +85,40 @@
   <xacro:gazebo_wheel ref="left_front_wheel" />
   <xacro:gazebo_wheel ref="left_back_wheel" />
+  <!--IMU : link, joint, sensor  -->
+<link name="imu_link">
+  <inertial>
+    <mass value="0.001"/>
+    <origin rpy="0 0 0" xyz="0 0 0"/>
+    <inertia ixx="0.0001" ixy="0" ixz="0" iyy="0.000001" iyz="0" izz="0.0001"/>
+  </inertial>
+  <visual>
+    <origin rpy="0 0 0" xyz="0 0 0"/>
+    <geometry>
+      <box size="0.01 0.01 0.01"/>
+    </geometry>
+  </visual>
+  <collision>
+    <origin rpy="0 0 0" xyz="0 0 0"/>
+    <geometry>
+      <box size="0.01 0.01 0.01"/>
+    </geometry>
+  </collision>
+</link>
+<joint name="imu_joint" type="fixed">
+  <axis xyz="1 0 0"/>
+  <origin xyz="0 0 0.105"/>
+  <parent link="base_link"/>
+  <child link="imu_link"/>
+</joint>
+<gazebo>
+    <plugin name="imu_plugin" filename="libgazebo_ros_imu.so">
+      <alwaysOn>true</alwaysOn>
+      <bodyName>imu_link</bodyName>
+      <topicName>imu</topicName>
+      <serviceName>imu_service</serviceName>
+      <gaussianNoise>0.0</gaussianNoise>
+      <updateRate>20.0</updateRate>
+    </plugin>
+  </gazebo>
   <!-- Gazebo plugin for ROS Control -->
   <gazebo>

Commit message: added an urdf link that is positioned at front of the robot

File: ros/src/robot_simulation/urdf/robot_simulation.xacro (robot description, xacro)
@@ -69,4 +69,30 @@
     </collision>
   </link>
+  <link name="front_mark">
+    <inertial>
+      <mass value="1"/>
+      <inertia ixx="1.0" ixy="0.0" ixz="0.0" iyy="1.0" iyz="0.0" izz="1.0"/>
+    </inertial>
+    <visual>
+        <origin xyz="0.0 0.0 0.0" rpy="0 0 0"/>
+        <geometry>
+            <cylinder radius="0.05" length="0.08"/>
+        </geometry>
+    </visual>
+    <collision>
+        <origin xyz="0.0 0.0 0.0" rpy="0 0 0"/>
+        <geometry>
+            <cylinder radius="0.05" length="0.08"/>
+        </geometry>
+    </collision>
+  </link>
+  <joint name="front_mark_joint" type="fixed">
+    <origin xyz="0.2 0.0 0.15" rpy="0.0 0.0 0.0"/>
+    <parent link="base_link"/>
+    <child link="front_mark"/>
+  </joint>
+  <gazebo reference="front_mark">
+      <material>Gazebo/Black</material>
+    </gazebo>
   <xacro:wheel_description name="right_front_wheel" />
   <xacro:wheel_description name="right_back_wheel" />
